File: Placa Digital.kicad_pcb (KiCad board)
At the start: 2 copper layers, 60 x 60 mm, 11 parts, among them J1 SALIDAS, J2 HMI, J4 ENTRADAS, U1 ESP32-DEVKITC-32D, U2 Alimentación

Commit message: Version V1 (Clearence)
Parts:
- U1: footprint LIB_ESP32-DevKitC:DIP2600W100P254L5400H500Q38N -> CEDCp:MODULE_ESP32-DEVKITC-32D
- moved U1 2.29 mm to (142.8, 85.4)
Routing:
- net /fromMicroC_DACI2C_SCL: track 85.4 -> 74.7 mm, vias 0 -> 2
- net /toMicroC_OverVoltageSignal: track 63.7 -> 72.4 mm
- net /toMicroC_ADC_BUSY: track 14.3 -> 22.6 mm
