File: Placa Digital.kicad_pcb (KiCad board)
At the start: 2 copper layers, 60 x 60 mm, 11 parts, among them J1 SALIDAS, J2 HMI, J4 ENTRADAS, U1 ESP32-DEVKITC-32D, U2 Alimentación

Commit message: Last version
Parts:
- added H1: MountingHole, MountingHole:MountingHole_2.2mm_M2_Pad_Via, F.Cu at (38.2, 133.0)
- added H1: MountingHole, MountingHole:MountingHole_2.2mm_M2_Pad_Via, F.Cu at (222.4, 133.2)
- added H1: MountingHole, MountingHole:MountingHole_2.2mm_M2_Pad_Via, F.Cu at (38.7, 25.3)
- added H1: MountingHole, MountingHole:MountingHole_2.2mm_M2_Pad_Via, F.Cu at (222.4, 25.3)
- added H2: MountingHole, MountingHole:MountingHole_2.2mm_M2_Pad_Via, F.Cu at (272.4, 25.3)
- added H2: MountingHole, MountingHole:MountingHole_2.2mm_M2_Pad_Via, F.Cu at (272.4, 133.2)
- added H2: MountingHole, MountingHole:MountingHole_2.2mm_M2_Pad_Via, F.Cu at (88.2, 133.0)
- added H2: MountingHole, MountingHole:MountingHole_2.2mm_M2_Pad_Via, F.Cu at (88.7, 25.3)
- added H3: MountingHole, MountingHole:MountingHole_2.2mm_M2_Pad_Via, F.Cu at (272.4, 183.2)
- added H3: MountingHole, MountingHole:MountingHole_2.2mm_M2_Pad_Via, F.Cu at (88.2, 183.0)
- added H3: MountingHole, MountingHole:MountingHole_2.2mm_M2_Pad_Via, F.Cu at (88.7, 75.3)
- added H3: MountingHole, MountingHole:MountingHole_2.2mm_M2_Pad_Via, F.Cu at (272.4, 75.3)
- added H4: MountingHole, MountingHole:MountingHole_2.2mm_M2_Pad_Via, F.Cu at (38.7, 75.3)
- added H4: MountingHole, MountingHole:MountingHole_2.2mm_M2_Pad_Via, F.Cu at (38.2, 183.0)
- added H4: MountingHole, MountingHole:MountingHole_2.2mm_M2_Pad_Via, F.Cu at (222.4, 75.3)
- added H4: MountingHole, MountingHole:MountingHole_2.2mm_M2_Pad_Via, F.Cu at (222.4, 183.2)
- added J1: SALIDAS, Connector_PinHeader_2.54mm:PinHeader_1x08_P2.54mm_Vertical, F.Cu at (267.4, 138.3)
- added J1: SALIDAS, Connector_PinHeader_2.54mm:PinHeader_1x08_P2.54mm_Vertical, F.Cu at (267.4, 30.4)
- added J1: SALIDAS, Connector_PinHeader_2.54mm:PinHeader_1x08_P2.54mm_Vertical, F.Cu at (83.7, 30.4)
- added J1: SALIDAS, Connector_PinHeader_2.54mm:PinHeader_1x08_P2.54mm_Vertical, F.Cu at (83.2, 138.1)
- added J2: HMI, Connector_PinHeader_2.54mm:PinHeader_1x08_P2.54mm_Vertical, F.Cu at (83.2, 161.0)
- added J2: HMI, Connector_PinHeader_2.54mm:PinHeader_1x08_P2.54mm_Vertical, F.Cu at (267.4, 161.2)
- added J2: HMI, Connector_PinHeader_2.54mm:PinHeader_1x08_P2.54mm_Vertical, F.Cu at (267.4, 53.3)
- added J2: HMI, Connector_PinHeader_2.54mm:PinHeader_1x08_P2.54mm_Vertical, F.Cu at (83.7, 53.3)
- added J4: ENTRADAS, Connector_PinHeader_2.54mm:PinHeader_1x10_P2.54mm_Vertical, F.Cu at (226.4, 141.4)
- added J4: ENTRADAS, Connector_PinHeader_2.54mm:PinHeader_1x10_P2.54mm_Vertical, F.Cu at (226.4, 33.5)
- added J4: ENTRADAS, Connector_PinHeader_2.54mm:PinHeader_1x10_P2.54mm_Vertical, F.Cu at (42.7, 33.5)
- added J4: ENTRADAS, Connector_PinHeader_2.54mm:PinHeader_1x10_P2.54mm_Vertical, F.Cu at (42.2, 141.2)
- added REF**: OSHW-Logo_5.7x6mm_SilkScreen, Symbol:OSHW-Logo_5.7x6mm_SilkScreen, F.Cu at (88.2, 175.0)
- added REF**: OSHW-Logo_5.7x6mm_SilkScreen, Symbol:OSHW-Logo_5.7x6mm_SilkScreen, F.Cu at (88.7, 67.3)
- added REF**: OSHW-Logo_5.7x6mm_SilkScreen, Symbol:OSHW-Logo_5.7x6mm_SilkScreen, F.Cu at (272.4, 67.3)
- added REF**: KiCad-Logo2_5mm_SilkScreen, Symbol:KiCad-Logo2_5mm_SilkScreen, F.Cu at (63.7, 48.3)
- added REF**: KiCad-Logo2_5mm_SilkScreen, Symbol:KiCad-Logo2_5mm_SilkScreen, F.Cu at (247.4, 156.2)
- added REF**: KiCad-Logo2_5mm_SilkScreen, Symbol:KiCad-Logo2_5mm_SilkScreen, F.Cu at (247.4, 48.3)
- added REF**: KiCad-Logo2_5mm_SilkScreen, Symbol:KiCad-Logo2_5mm_SilkScreen, F.Cu at (63.2, 156.0)
- added REF**: OSHW-Logo_5.7x6mm_SilkScreen, Symbol:OSHW-Logo_5.7x6mm_SilkScreen, F.Cu at (272.4, 175.2)
- added U1: ESP32-DEVKITC-32D, CEDCp:MODULE_ESP32-DEVKITC-32D, F.Cu at (63.0, 159.4)
- added U1: ESP32-DEVKITC-32D, CEDCp:MODULE_ESP32-DEVKITC-32D, F.Cu at (63.5, 51.7)
- added U1: ESP32-DEVKITC-32D, CEDCp:MODULE_ESP32-DEVKITC-32D, F.Cu at (247.1, 51.7)
- added U1: ESP32-DEVKITC-32D, CEDCp:MODULE_ESP32-DEVKITC-32D, F.Cu at (247.1, 159.6)
- added U2: Alimentación, CEDCp:Bornera_1x2, F.Cu at (225.4, 172.2)
- added U2: Alimentación, CEDCp:Bornera_1x2, F.Cu at (225.4, 64.3)
- added U2: Alimentación, CEDCp:Bornera_1x2, F.Cu at (41.2, 172.0)
- added U2: Alimentación, CEDCp:Bornera_1x2, F.Cu at (41.7, 64.3)
- moved J4 10.4 mm to (132.2, 69.3)
- moved H1 10.4 mm to (128.2, 61.1)
- moved H2 10.4 mm to (178.2, 61.1)
- moved H3 10.4 mm to (178.2, 111.1)
- moved H4 10.4 mm to (128.2, 111.1)
- moved J1 10.4 mm to (173.2, 66.2)
- moved J2 10.4 mm to (173.2, 89.1)
- moved REF** 10.4 mm to (153.2, 84.1)
- moved REF** 10.4 mm to (178.2, 103.1)
- moved U1 10.4 mm to (152.9, 87.5)
- moved U2 10.4 mm to (131.2, 100.1)
Routing:
- net /fromMicroC_DACI2C_SCL: track 74.7 -> 373.3 mm, vias 2 -> 10
- net /toMicroC_OverVoltageSignal: track 72.4 -> 362.0 mm, vias 2 -> 10
- net /fromMicroC_ADC_CONV: track 69.3 -> 346.3 mm
- net /fromMicroC_ADC_RST: track 67.4 -> 336.9 mm
- net /fromMicroC_ADC_RD: track 64.9 -> 324.7 mm
- net /fromMicroC_DACI2C_SDA: track 56.0 -> 280.1 mm
- net /toMicroC_ADC_BUSY: track 22.6 -> 113.2 mm
- net +5V: track 15.5 -> 77.4 mm
- net /toMicroC_EncoderSignalA: track 14.6 -> 73.1 mm
- net /toMicroC_EncoderSignalB: track 14.1 -> 70.5 mm
- net /fromMicroC_DisplaySCLK: track 13.8 -> 69.2 mm
- net /toMicroC_EncoderButton: track 13.7 -> 68.4 mm
- net /fromMicroC_DisplaySID: track 13.1 -> 65.7 mm
- net /fromMicroC_A6841CLK1: track 11.4 -> 57.1 mm
- net /fromMicroC_A6841SerialDataIN: track 11.4 -> 57.1 mm
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Other:
- board size 60 x 60 mm -> 244.1 x 168 mm
